Commit message: Update mecanum.xacro

File: src/mentorpi_description/urdf/mecanum.xacro (robot description, xacro)
@@ -219,5 +219,5 @@
     <parent link="base_link"/>
     <child link="wheel_right_front_link"/>
-    <axis xyz="0 -1 0"/>
+    <axis xyz="0 1 0"/>
     <limit lower="0" upper="0" effort="0" velocity="0"/>
   </joint>
@@ -251,5 +251,5 @@
     <parent link="base_link"/>
     <child link="wheel_right_back_link"/>
-    <axis xyz="0 -1 0"/>
+    <axis xyz="0 1 0"/>
     <limit lower="0" upper="0" effort="0" velocity="0"/>
   </joint>
