Commit message: Update gripper.urdf.xacro

File: src/mentorpi_description/urdf/gripper.urdf.xacro (robot description, xacro)
@@ -32,5 +32,5 @@
     <parent link="gripper_link"/>
     <child link="r_link"/>
-    <axis xyz="0.999999784828379 0.000360574512731351 -0.000548023007084987"/>
+    <axis xyz="-0.999999784828379 -0.000360574512731351 0.000548023007084987"/>
     <limit lower="-1.57" upper="1.57" effort="1000" velocity="10"/>
   </joint>
@@ -68,5 +68,5 @@
     <mimic
       joint="r_joint"
-      multiplier="-1"
+      multiplier="1"
       offset="0" />
   </joint>
@@ -104,5 +104,5 @@
     <mimic
       joint="r_joint"
-      multiplier="-1"
+      multiplier="1"
       offset="0" />
   </joint>
@@ -140,5 +140,5 @@
     <mimic
       joint="r_joint"
-      multiplier="1"
+      multiplier="-1"
       offset="0" />
   </joint>
@@ -176,5 +176,5 @@
     <mimic
       joint="r_joint"
-      multiplier="1"
+      multiplier="-1"
       offset="0" />
   </joint>
@@ -212,5 +212,5 @@
     <mimic
       joint="r_joint"
-      multiplier="-1"
+      multiplier="1"
       offset="0" />
   </joint>
